File: amurNutzlast/clock.kicad_sch (KiCad schematic)
At the start: 2 parts, among them X1 SG-7050CAN

Commit message: layout start
Parts:
- C18: footprint (none) -> Capacitor_SMD:C_0603_1608Metric
Changed lines of the file:
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@@
       (effects (font (size 1.27 1.27)) (justify left))
     )
-    (property "Footprint" "" (at 129.54 83.82 0)
+    (property "Footprint" "Capacitor_SMD:C_0603_1608Metric" (at 129.54 83.82 0)
       (effects (font (size 1.27 1.27)) hide)
     )
