File: amurNutzlast/flash.kicad_sch (KiCad schematic)
At the start: 6 parts, among them U3 N25Q032A13ESQC40F

Commit message: finisched design schematics + pdf
Parts:
- removed U3: N25Q032A13ESQC40F, Package_SO:SOP-8_3.9x4.9mm_P1.27mm, symbol Memory_Flash:W25Q32JVSS
- added U6: W25Q128JVS, Package_SO:SOIC-8_5.23x5.23mm_P1.27mm, symbol Memory_Flash:W25Q128JVS
Connections:
- net +3.3V: now also U6.8 (VCC)
- net CLK: now also U6.6 (CLK)
- net GND: now also U6.4 (GND)
- net MISO: now also U6.2 (DO(IO1))
- net MOSI: now also U6.5 (DI(IO0))
- net SS: now also U6.1 (~{CS})
- net at R16.2: now also U6.3 (IO2)
- net at R17.2: now also U6.7 (IO3)
Changed lines of the file:
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@@
+    )
+  )
+  (symbol (lib_id "Memory_Flash:W25Q128JVS") (at 134.62 88.9 0) (unit 1)
+    (in_bom yes) (on_board yes) (dnp no) (fields_autoplaced)
+    (property "Reference" "U6" (at 143.51 87.63 0)
+      (effects (font (size 1.27 1.27)) (justify left))
+    )
+    (property "Value" "W25Q128JVS" (at 143.51 90.17 0)
+      (effects (font (size 1.27 1.27)) (justify left))
+    )
+    (property "Footprint" "Package_SO:SOIC-8_5.23x5.23mm_P1.27mm" (at 134.62 88.9 0)
+      (effects (font (size 1.27 1.27)) hide)
+    )
+    (property "Datasheet" "http://www.winbond.com/resource-files/w25q128jv_dtr%20revc%2003272018%20plus.pdf" (at 134.62 88.9 0)
+      (effects (font (size 1.27 1.27)) hide)
+    )
+    (pin "1")
+    (pin "2")
+    (pin "3")
+    (pin "4")
+    (pin "5")
+    (pin "6")
+    (pin "7")
+    (pin "8")
+    (instances
+      (project "amurNutzlast"
+        (path "/81bb76b1-eb1b-4eda-9d04-3f9c2ab6907c/5a1048a1-8aad-441a-9502-b80402a1bae3"
+          (reference "U6") (unit 1)
+        )
+      )
     )
   )
@@
         )
       )
-    )
-  )
-  (symbol (lib_id "Memory_Flash:W25Q32JVSS") (at 134.62 88.9 0) (unit 1)
-    (in_bom yes) (on_board yes) (dnp no) (fields_autoplaced)
-    (property "Reference" "U3" (at 143.51 87.63 0)
-      (effects (font (size 1.27 1.27)) (justify left))
-    )
-    (property "Value" "N25Q032A13ESQC40F" (at 143.51 90.17 0)
-      (effects (font (size 1.27 1.27)) (justify left))
-    )
-    (property "Footprint" "Package_SO:SOP-8_3.9x4.9mm_P1.27mm" (at 134.62 88.9 0)
-      (effects (font (size 1.27 1.27)) hide)
-    )
-    (property "Datasheet" "https://www.mouser.de/ProductDetail/Alliance-Memory/N25Q032A13ESC40F?qs=W%2FMpXkg%252BdQ70%2FmLJsMq3Ww%3D%3D" (at 134.62 88.9 0)
-      (effects (font (size 1.27 1.27)) hide)
-    )
-    (pin "1")
-    (pin "2")
-    (pin "3")
-    (pin "4")
-    (pin "5")
-    (pin "6")
-    (pin "7")
-    (pin "8")
-    (instances
-      (project "amurNutzlast"
-        (path "/81bb76b1-eb1b-4eda-9d04-3f9c2ab6907c/5a1048a1-8aad-441a-9502-b80402a1bae3"
-          (reference "U3") (unit 1)
-        )
-      )

Commit message: layout start
Parts:
- C24: footprint (none) -> Capacitor_SMD:C_0603_1608Metric
- R15, R16, R17, R18: footprint (none) -> Resistor_SMD:R_0603_1608Metric
Changed lines of the file:
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@@
       (effects (font (size 1.27 1.27)) (justify left))
     )
-    (property "Footprint" "" (at 116.84 68.58 0)
+    (property "Footprint" "Resistor_SMD:R_0603_1608Metric" (at 116.84 68.58 0)
       (effects (font (size 1.27 1.27)) hide)
     )
@@
       (effects (font (size 1.27 1.27)) (justify left))
     )
-    (property "Footprint" "" (at 93.98 68.58 0)
+    (property "Footprint" "Resistor_SMD:R_0603_1608Metric" (at 93.98 68.58 0)
       (effects (font (size 1.27 1.27)) hide)
     )
@@
       (effects (font (size 1.27 1.27)) (justify left))
     )
-    (property "Footprint" "" (at 86.36 68.58 0)
+    (property "Footprint" "Resistor_SMD:R_0603_1608Metric" (at 86.36 68.58 0)
       (effects (font (size 1.27 1.27)) hide)
     )
@@
       (effects (font (size 1.27 1.27)) (justify left))
     )
-    (property "Footprint" "" (at 104.14 68.58 0)
+    (property "Footprint" "Resistor_SMD:R_0603_1608Metric" (at 104.14 68.58 0)
       (effects (font (size 1.27 1.27)) hide)
     )
@@
       (effects (font (size 1.27 1.27)) (justify left))
     )
-    (property "Footprint" "" (at 149.86 71.12 0)
-      (effects (font (size 1.27 1.27)) hide)
-    )
+    (property "Footprint" "Capacitor_SMD:C_0603_1608Metric" (at 149.86 71.12 0)
+      (effects (font (size 1.27 1.27)) hide)
+    )
