File: amurNutzlast/usb.kicad_sch (KiCad schematic)
At the start: 4 parts, among them J2 USB_A

Commit message: ftdi layout continuation
Changed lines of the file:
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@@
     (stroke (width 0) (type default))
+  )
+  (label "-" (at 109.22 109.22 0) (fields_autoplaced)
+    (effects (font (size 1.27 1.27)) (justify left bottom))
+  )
+  (label "+" (at 109.22 106.68 0) (fields_autoplaced)
+    (effects (font (size 1.27 1.27)) (justify left bottom))
   )
   (hierarchical_label "DP" (shape output) (at 114.3 106.68 0) (fields_autoplaced)
