File: amurNutzlast/amurNutzlast.kicad_sch (KiCad schematic)
At the start: 6 parts, among them J1 Conn_01x08, J3 Conn_01x02, J4 Conn_01x08, J5 Conn_01x07, J7 Conn_01x07, J8 Conn_01x20

Commit message: started FPGA
Parts:
- removed J3: Conn_01x02, LED_SMD:LED_0603_1608Metric, symbol Connector_Generic:Conn_01x02
Other:
- note removed: "jumper to supply input power to the FPGA"
Changed lines of the file:
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@@
-    (stroke (width 0) (type default))
-  )
-  (wire (pts (xy 68.58 20.32) (xy 68.58 27.94))
     (stroke (width 0) (type default))
   )
@@
     (stroke (width 0) (type default))
   )
-  (wire (pts (xy 60.96 25.4) (xy 55.88 25.4))
-    (stroke (width 0) (type default))
-  )
   (wire (pts (xy 142.24 68.58) (xy 157.48 68.58))
     (stroke (width 0) (type default))
@@
     (stroke (width 0) (type default))
   )
-  (wire (pts (xy 55.88 27.94) (xy 68.58 27.94))
-    (stroke (width 0) (type default))
-  )
   (wire (pts (xy 111.76 96.52) (xy 114.3 96.52))
     (stroke (width 0) (type default))
@@
     (stroke (width 0) (type default))
   )
-  (wire (pts (xy 60.96 20.32) (xy 60.96 25.4))
-    (stroke (width 0) (type default))
-  )
   (wire (pts (xy 193.04 81.28) (xy 193.04 73.66))
     (stroke (width 0) (type default))
@@
   (wire (pts (xy 137.16 30.48) (xy 137.16 66.04))
     (stroke (width 0) (type default))
-  )
-  (text "jumper to supply input\npower to the FPGA" (at 73.66 22.86 0)
-    (effects (font (size 1.27 1.27)) (justify left bottom))
   )
   (label "ICE_CDONE" (at 116.84 60.96 0) (fields_autoplaced)
@@
         (path "/81bb76b1-eb1b-4eda-9d04-3f9c2ab6907c"
           (reference "J7") (unit 1)
-        )
-      )
-    )
-  )
-  (symbol (lib_id "power:VBUS") (at 60.96 20.32 0) (unit 1)
-    (in_bom yes) (on_board yes) (dnp no) (fields_autoplaced)
-    (property "Reference" "#PWR056" (at 60.96 24.13 0)
-      (effects (font (size 1.27 1.27)) hide)
-    )
-    (property "Value" "VBUS" (at 60.96 15.24 0)
-      (effects (font (size 1.27 1.27)))
-    )
-    (property "Footprint" "" (at 60.96 20.32 0)
-      (effects (font (size 1.27 1.27)) hide)
-    )
-    (property "Datasheet" "" (at 60.96 20.32 0)
-      (effects (font (size 1.27 1.27)) hide)
-    )
-    (pin "1")
-    (instances
-      (project "amurNutzlast"
-        (path "/81bb76b1-eb1b-4eda-9d04-3f9c2ab6907c"
-          (reference "#PWR056") (unit 1)
-        )
-      )
-    )
-  )
-  (symbol (lib_id "power:+5V") (at 68.58 20.32 0) (unit 1)
-    (in_bom yes) (on_board yes) (dnp no) (fields_autoplaced)
-    (property "Reference" "#PWR087" (at 68.58 24.13 0)
-      (effects (font (size 1.27 1.27)) hide)
-    )
-    (property "Value" "+5V" (at 68.58 15.24 0)
-      (effects (font (size 1.27 1.27)))
-    )
-    (property "Footprint" "" (at 68.58 20.32 0)
-      (effects (font (size 1.27 1.27)) hide)
-    )
-    (property "Datasheet" "" (at 68.58 20.32 0)
-      (effects (font (size 1.27 1.27)) hide)
-    )
-    (pin "1")
-    (instances
-      (project "amurNutzlast"
-        (path "/81bb76b1-eb1b-4eda-9d04-3f9c2ab6907c"
-          (reference "#PWR087") (unit 1)
         )
       )
@@
         )
       )
-    )
-  )
-  (symbol (lib_id "Connector_Generic:Conn_01x02") (at 50.8 27.94 180) (unit 1)
-    (in_bom yes) (on_board yes) (dnp no) (fields_autoplaced)
-    (property "Reference" "J3" (at 50.8 19.05 0)
-      (effects (font (size 1.27 1.27)))
-    )
-    (property "Value" "Conn_01x02" (at 50.8 21.59 0)
-      (effects (font (size 1.27 1.27)))
-    )
-    (property "Footprint" "LED_SMD:LED_0603_1608Metric" (at 50.8 27.94 0)
-      (effects (font (size 1.27 1.27)) hide)
-    )
-    (property "Datasheet" "~" (at 50.8 27.94 0)
-      (effects (font (size 1.27 1.27)) hide)
-    )
-    (pin "1")
-    (pin "2")
-    (instances
-      (project "amurNutzlast"
-        (path "/81bb76b1-eb1b-4eda-9d04-3f9c2ab6907c"
-          (reference "J3") (unit 1)
-        )
-      )

Commit message: placement finished
Parts:
- removed J1: Conn_01x08, Connector_PinHeader_2.54mm:PinHeader_2x04_P2.54mm_Vertical, symbol Connector_Generic:Conn_01x08
- added J1: Conn_01x06, Connector_PinHeader_2.54mm:PinHeader_2x03_P2.54mm_Vertical, symbol Connector_Generic:Conn_01x06
Connections:
- net ICE_CDONE: now also J1.2 (Pin_2)
- net ICE_CREST: now also J1.1 (Pin_1)
- net MISO: now also J1.3 (Pin_3)
- net MOSI: now also J1.4 (Pin_4)
- net SCL: now also J1.5 (Pin_5)
- net SS: now also J1.6 (Pin_6)
Changed lines of the file:
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@@
-    (stroke (width 0) (type default))
-  )
-  (wire (pts (xy 152.4 73.66) (xy 157.48 73.66))
     (stroke (width 0) (type default))
   )
@@
     (stroke (width 0) (type default))
   )
-  (wire (pts (xy 147.32 81.28) (xy 152.4 81.28))
-    (stroke (width 0) (type default))
-  )
   (wire (pts (xy 111.76 63.5) (xy 132.08 63.5))
     (stroke (width 0) (type default))
@@
     (stroke (width 0) (type default))
   )
-  (wire (pts (xy 154.94 76.2) (xy 154.94 81.28))
-    (stroke (width 0) (type default))
-  )
   (wire (pts (xy 147.32 35.56) (xy 147.32 71.12))
     (stroke (width 0) (type default))
@@
     (stroke (width 0) (type default))
   )
-  (wire (pts (xy 147.32 78.74) (xy 147.32 81.28))
-    (stroke (width 0) (type default))
-  )
   (wire (pts (xy 132.08 139.7) (xy 132.08 154.94))
     (stroke (width 0) (type default))
@@
     (stroke (width 0) (type default))
   )
-  (wire (pts (xy 154.94 76.2) (xy 157.48 76.2))
-    (stroke (width 0) (type default))
-  )
   (wire (pts (xy 154.94 144.78) (xy 137.16 144.78))
     (stroke (width 0) (type default))
@@
     (stroke (width 0) (type default))
   )
-  (wire (pts (xy 152.4 81.28) (xy 152.4 73.66))
-    (stroke (width 0) (type default))
-  )
   (wire (pts (xy 137.16 30.48) (xy 137.16 66.04))
     (stroke (width 0) (type default))
@@
   (label "MISO" (at 116.84 63.5 0) (fields_autoplaced)
     (effects (font (size 1.27 1.27)) (justify left bottom))
-  )
-  (symbol (lib_id "power:+3.3V") (at 147.32 78.74 0) (unit 1)
-    (in_bom yes) (on_board yes) (dnp no) (fields_autoplaced)
-    (property "Reference" "#PWR045" (at 147.32 82.55 0)
-      (effects (font (size 1.27 1.27)) hide)
-    )
-    (property "Value" "+3.3V" (at 147.32 73.66 0)
-      (effects (font (size 1.27 1.27)))
-    )
-    (property "Footprint" "" (at 147.32 78.74 0)
-      (effects (font (size 1.27 1.27)) hide)
-    )
-    (property "Datasheet" "" (at 147.32 78.74 0)
-      (effects (font (size 1.27 1.27)) hide)
-    )
-    (pin "1")
-    (instances
-      (project "amurNutzlast"
-        (path "/81bb76b1-eb1b-4eda-9d04-3f9c2ab6907c"
-          (reference "#PWR045") (unit 1)
-        )
-      )
-    )
   )
   (symbol (lib_id "Connector_Generic:Conn_01x08") (at 180.34 68.58 180) (unit 1)
@@
     )
   )
-  (symbol (lib_id "Connector_Generic:Conn_01x08") (at 162.56 66.04 0) (unit 1)
+  (symbol (lib_id "Connector_Generic:Conn_01x06") (at 162.56 63.5 0) (unit 1)
+    (in_bom yes) (on_board yes) (dnp no) (fields_autoplaced)
+    (property "Reference" "J1" (at 165.1 63.5 0)
+      (effects (font (size 1.27 1.27)) (justify left))
+    )
+    (property "Value" "Conn_01x06" (at 165.1 66.04 0)
+      (effects (font (size 1.27 1.27)) (justify left))
+    )
+    (property "Footprint" "Connector_PinHeader_2.54mm:PinHeader_2x03_P2.54mm_Vertical" (at 162.56 63.5 0)
+      (effects (font (size 1.27 1.27)) hide)
+    )
+    (property "Datasheet" "~" (at 162.56 63.5 0)
+      (effects (font (size 1.27 1.27)) hide)
+    )
+    (pin "1")
+    (pin "2")
+    (pin "3")
+    (pin "4")
+    (pin "5")
+    (pin "6")
+    (instances
+      (project "amurNutzlast"
+        (path "/81bb76b1-eb1b-4eda-9d04-3f9c2ab6907c"
+          (reference "J1") (unit 1)
+        )
+      )
+    )
+  )
+  (symbol (lib_id "Connector_Generic:Conn_01x07") (at 180.34 144.78 180) (unit 1)
     (in_bom yes) (on_board yes) (dnp no)
-    (property "Reference" "J1" (at 162.56 50.8 0)
-      (effects (font (size 1.27 1.27)) (justify left))
-    )
-    (property "Value" "Conn_01x08" (at 157.48 53.34 0)
-      (effects (font (size 1.27 1.27)) (justify left))
-    )
-    (property "Footprint" "Connector_PinHeader_2.54mm:PinHeader_2x04_P2.54mm_Vertical" (at 162.56 66.04 0)
-      (effects (font (size 1.27 1.27)) hide)
-    )
-    (property "Datasheet" "~" (at 162.56 66.04 0)
+    (property "Reference" "J5" (at 180.34 129.54 0)
+      (effects (font (size 1.27 1.27)))
+    )
+    (property "Value" "Conn_01x07" (at 180.34 132.08 0)
+      (effects (font (size 1.27 1.27)))
+    )
+    (property "Footprint" "Connector_PinHeader_2.54mm:PinHeader_1x07_P2.54mm_Vertical" (at 180.34 144.78 0)
+      (effects (font (size 1.27 1.27)) hide)
+    )
+    (property "Datasheet" "~" (at 180.34 144.78 0)
       (effects (font (size 1.27 1.27)) hide)
     )
@@
     (pin "6")
     (pin "7")
-    (pin "8")
-    (instances
-      (project "amurNutzlast"
-        (path "/81bb76b1-eb1b-4eda-9d04-3f9c2ab6907c"
-          (reference "J1") (unit 1)
-        )
-      )
-    )
-  )
-  (symbol (lib_id "Connector_Generic:Conn_01x07") (at 180.34 144.78 180) (unit 1)
-    (in_bom yes) (on_board yes) (dnp no)
-    (property "Reference" "J5" (at 180.34 129.54 0)
-      (effects (font (size 1.27 1.27)))
-    )
-    (property "Value" "Conn_01x07" (at 180.34 132.08 0)
-      (effects (font (size 1.27 1.27)))
-    )
-    (property "Footprint" "Connector_PinHeader_2.54mm:PinHeader_1x07_P2.54mm_Vertical" (at 180.34 144.78 0)
-      (effects (font (size 1.27 1.27)) hide)
-    )
-    (property "Datasheet" "~" (at 180.34 144.78 0)
-      (effects (font (size 1.27 1.27)) hide)
-    )
-    (pin "1")
-    (pin "2")
-    (pin "3")
-    (pin "4")
-    (pin "5")
-    (pin "6")
-    (pin "7")
     (instances
       (project "amurNutzlast"
@@
         )
       )
-    )
-  )
-  (symbol (lib_id "power:GND") (at 154.94 81.28 0) (unit 1)
-    (in_bom yes) (on_board yes) (dnp no) (fields_autoplaced)
-    (property "Reference" "#PWR046" (at 154.94 87.63 0)
-      (effects (font (size 1.27 1.27)) hide)
-    )
-    (property "Value" "GND" (at 154.94 86.36 0)
-      (effects (font (size 1.27 1.27)))
-    )
-    (property "Footprint" "" (at 154.94 81.28 0)
-      (effects (font (size 1.27 1.27)) hide)
-    )
-    (property "Datasheet" "" (at 154.94 81.28 0)
-      (effects (font (size 1.27 1.27)) hide)
-    )
-    (pin "1")
-    (instances
-      (project "amurNutzlast"
-        (path "/81bb76b1-eb1b-4eda-9d04-3f9c2ab6907c"
-          (reference "#PWR046") (unit 1)
-        )
-      )

Commit message: finished pcb
Parts:
- removed J4: Conn_01x08, Connector_PinHeader_2.54mm:PinHeader_2x04_P2.54mm_Vertical, symbol Connector_Generic:Conn_01x08
- added H1, H2, H3, H5: MountingHole_Pad, MountingHole:MountingHole_2.5mm_Pad_Via, symbol Mechanical:MountingHole_Pad
- added J3: Conn_01x06, Connector_PinHeader_2.54mm:PinHeader_2x03_P2.54mm_Vertical, symbol Connector_Generic:Conn_01x06
Connections:
- net GND1: now also H2.1, H3.1
- net ICE_CREST: now also J1.4 (Pin_4); no longer J1.1 (Pin_1)
- net MISO: now also J1.1 (Pin_1); no longer J1.3 (Pin_3)
- net MOSI: now also J1.5 (Pin_5); no longer J1.4 (Pin_4)
- net SCL: now also J1.6 (Pin_6); no longer J1.5 (Pin_5)
- net SS: now also J1.3 (Pin_3); no longer J1.6 (Pin_6)
- net ftdi/ICE_CDONE: now also J3.3 (Pin_3)
- net ftdi/ICE_CLK: now also J3.2 (Pin_2)
- net ftdi/ICE_CREST: now also J3.1 (Pin_1)
- net ftdi/ICE_MISO: now also J3.6 (Pin_6)
- net ftdi/ICE_MOSI: now also J3.4 (Pin_4)
- net ftdi/ICE_SS: now also J3.5 (Pin_5)
- new net GND: H1.1, H5.1
Other:
- moved on the sheet: J1
